File: PB01 - Hardware/HW03 - Placa de da ECU1 Telemetria/ecu1_telemetria.sch (EAGLE design)
At the start: 26 parts, among them IC1 LM358N, Q2 16MHz, X1 22-23-2021, X5 22-23-2021, X6 22-23-2021, X8 22-23-2031

Commit message: ECU1
Parts:
- removed IC1: LM358N, linear3:LM358N
- added IC2: LM324N, linear:LM324N
Connections:
- removed net N$4: IC1B.-IN, IC1B.OUT, R4.1
- new net N$3: IC2A.-IN, IC2A.OUT, R4.1
- net +5V: now also IC2P.V+; no longer IC1P.V+
- net GND: now also IC2P.V-; no longer IC1P.V-
- net N$7: now also IC2A.+IN; no longer IC1B.+IN
- net N$8: now also IC2B.+IN; no longer IC1A.+IN
- net PA10: now also IC2B.-IN, IC2B.OUT; no longer IC1A.-IN, IC1A.OUT
Other:
- moved on the sheet: C2, C4
