File: PB01 - Hardware/HW03 - Placa de ECU1 Telemetria/ecu1_telemetria.sch (EAGLE design)
At the start: 30 parts, among them IC2 LM324N, Q2 16MHz, X1 22-23-2021, X2 22-23-2031, X3 22-23-2031, X4 22-23-2071, X5 22-23-2021, X6 22-23-2021

Commit message: TE#LEMETRIA
Parts:
- removed X5, X6: 22-23-2021, con-molex:22-23-2021
- added X7: FORÇA, con-molex:22-23-2031
- C2: device capacitor-wima:C2,5-3 -> capacitor-wima:C5/2.5
- X1: value 22-23-2021 -> RPM
- X2: value 22-23-2031 -> COMB 1
- X3: value 22-23-2031 -> COMB 2
- X4: value 22-23-2071 -> MODULE CAN
- renumbered OK1 to OPTO, Q2 to CRISTAL, S1 to BOTÃO
Connections:
- net +12V: now also X7-2.S; no longer X6-1.S
- net +5V: now also X7-1.S; no longer X5-1.S
- net COMB2_OUT: now also ZIC1.(T0)PD4
- net GND: now also X7-3.S; no longer X5-2.S, X6-2.S
