File: PB01 - Hardware/HW04 - Placa de ECU2 Telemetria/ecu2_telemetria.brd (EAGLE design)
At the start: 67.6 x 85.9 mm, 26 parts, among them IC2 LM324N, Q2 16MHz, X1 22-23-2021, X5 22-23-2021, X6 22-23-2021, X8 22-23-2031

Commit message: TE#LEMETRIA
Parts:
- removed C1, C4: 100nF, capacitor-wima:C5B2.5
- removed D5: 1N4004, diode:DO41-10
- removed D6: 3.3V, diode:DO34Z7
- removed IC2: LM324N, linear:DIL14
- removed OK1: PC817, optocoupler:DIL04
- removed Q2: 16MHz, special:QS
- removed R1, R2, R4, R8: 1k, resistor:0207/7
- removed R3: 10k, resistor:0207/7
- removed R7: 4.7KR, resistor:0207/7
- removed S1: (no value), switch-omron:B3F-10XX
- removed SV1: (no value), con-lstb:MA06-1
- removed X6: 22-23-2021, con-molex:22-23-2021
- removed X8: 22-23-2031, con-molex:22-23-2031
- added BOTÃO: (no value), switch-omron:B3F-10XX
- added C7, C8: 100nF, capacitor-wima:C5B2.5
- added CRISTAL: 16MHz, special:QS
- added D2, D3: 5.0V, diode:DO34Z7
- added IC1: LM358N, linear:DIL08
- added R10, R12: 1k, resistor:0207/7
- added R11, R9: 4.7KR, resistor:0207/7
- added X2: COMB 1, con-molex:22-23-2031
- added X3: COMB 2, con-molex:22-23-2031
- added X4: MODULE CAN, con-molex:22-23-2071
- added X7: FORÇA, con-molex:22-23-2031
- C2: device capacitor-wima:C2.5-3 -> capacitor-wima:C5B2.5
- X1: value 22-23-2021 -> DAC; device con-molex:22-23-2021 -> con-molex:22-23-2031
- X5: value 22-23-2021 -> 22-23-2041; device con-molex:22-23-2021 -> con-molex:22-23-2041
- moved SV8 131.6 mm to (158.4, -22.6), turned to 90 degrees
- moved X5 118.0 mm to (144.2, 24.0), turned to 0 degrees
- moved ZIC1 109.6 mm to (156.5, 6.00), turned to 270 degrees
- moved C6 95.3 mm to (144.9, -8.74), turned to 0 degrees
- moved C5 89.4 mm to (144.9, -3.77), turned to 0 degrees
- moved R5 89.3 mm to (122.9, 13.5), turned to 180 degrees
- moved C3 89.3 mm to (122.9, 24.9), turned to 180 degrees
- moved X1 71.5 mm to (133.2, 24.0), turned to 0 degrees
- moved C2 66.6 mm to (113.5, 25.0), turned to 180 degrees
Connections:
- removed net N$1: OK1.1, R1.2, R2.2
- removed net N$2: D5.C, R1.1, R2.1
- removed net N$7: IC2.3, OK1.3, R3.2
- removed net N$8: D6.C, IC2.5, R7.2
- removed net PA10: IC2.6, IC2.7, R8.1
- removed net RPM_GND: OK1.2, X1.2
- removed net RPM_IN: D5.A, X1.1
- removed net RPM_OUT: C1.2, R4.2, ZIC1.4
- removed net VEL_IN: R7.1, X8.2
- removed net VEL_OUT: C4.2, R8.2, ZIC1.5
- new net N$12: IC1.1, IC1.2, R10.1
- new net N$13: D3.C, IC1.5, R11.2
- new net N$14: IC1.6, IC1.7, R12.1
- new net N$5: D2.C, IC1.3, R9.2
- new net SCL: X5.3, ZIC1.28
- new net SDA: X5.4, ZIC1.27
- new net VEL1_IN: R9.1, X3.2
- new net VEL1_OUT: C7.2, R10.2, ZIC1.5
- new net VEL2_IN: R11.1, X2.2
- new net VEL2_OUT: C8.2, R12.2, ZIC1.4
- net +12V: now also X2.1, X3.1, X7.2; no longer X6.1, X8.1
- net +5V: now also IC1.4, X1.1, X4.7, X7.1; no longer IC2.4, OK1.4, SV1.5
- net GND: now also BOTÃO.1, BOTÃO.2, C7.1, C8.1, D2.A, D3.A, IC1.8, X1.2, X2.3, X3.3, X4.6, X7.3; no longer C1.1, C4.1, D6.A, IC2.11, R3.1, S1.1, S1.2, SV1.6, X6.2, X8.3
- net MISO: now also X4.4; no longer SV1.4
- net MOSI: now also X4.3; no longer SV1.3
- net N$3: now also X1.3, ZIC1.12; no longer IC2.1, IC2.2, R4.1
- net N$9: now also BOTÃO.3, BOTÃO.4; no longer S1.3, S1.4
- net SCK: now also X4.2; no longer SV1.2
- net SS: now also X4.5; no longer SV1.1
- net XTAL1: now also CRISTAL.2; no longer Q2.2
- net XTAL2: now also CRISTAL.1; no longer Q2.1
Routing:
- net +5V: track 94.9 -> 28.6 mm
- net IO8: track 44.2 -> 0.00 mm
- net IO9: track 31.3 -> 0.00 mm
- net VEL_OUT: track 21.6 -> 0.00 mm
- net XTAL1: track 9.81 -> 29.2 mm
- net RPM_GND: track 18.1 -> 0.00 mm
- net SCK: track 16.1 -> 0.00 mm
- net N$9: track 15.2 -> 0.00 mm
- net RPM_OUT: track 15.0 -> 0.00 mm
- net N$7: track 14.3 -> 0.00 mm
- net N$2: track 13.6 -> 0.00 mm
- net VEL2_IN: track 0.00 -> 12.4 mm
- net N$1: track 10.2 -> 0.00 mm
- net VEL_IN: track 10.1 -> 0.00 mm
- net XTAL2: track 9.82 -> 18.2 mm
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- added copper zone on layer 16, net MODULE_CAN
- added copper zone on layer 16, net N$1
- removed copper zone on layer 16, net GND
Other:
- board size 67.6 x 85.9 mm -> 326.4 x 201.8 mm
- board text added: "Design by: Matheus Torres Rocha"
- board text added: "Equipe ParahyBaja ECU1"

Commit message: TELEMETRIA
Parts:
- moved D2 11.1 mm to (119.8, 4.97)
- moved R9 11.1 mm to (123.8, 4.97)
- moved X3 11.1 mm to (113.0, 4.63)
- moved D3 11.0 mm to (120.0, -6.17)
- moved R11 11.0 mm to (124.0, -6.17)
- moved X2 11.0 mm to (113.3, -6.69)
- moved C8 9.95 mm to (145.0, 12.2)
- moved R12 9.26 mm to (144.9, 15.4)
- moved C7 9.09 mm to (144.9, 2.40)
- moved R10 9.09 mm to (144.9, 6.52)
- moved BOTÃO 0.38 mm to (122.8, 19.0), turned to 0 degrees
Routing:
- net +5V: track 28.6 -> 212.4 mm
- net N$3: track 0.00 -> 115.6 mm
- net N$9: track 0.00 -> 39.3 mm
- net +12V: track 0.00 -> 26.1 mm
- net N$13: track 0.00 -> 25.8 mm
- net SS: track 0.00 -> 24.3 mm
- net SCK: track 0.00 -> 24.1 mm
- net MISO: track 0.00 -> 20.3 mm
- net SCL: track 0.00 -> 17.1 mm
- net GND: track 0.00 -> 16.3 mm, vias 0 -> 2
- net MOSI: track 0.00 -> 15.9 mm
- net N$12: track 0.00 -> 15.6 mm
- net SDA: track 0.00 -> 14.6 mm
- net IO8: track 0.00 -> 14.5 mm
- net VEL1_OUT: track 0.00 -> 13.2 mm
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- added copper zone on layer 16, net GND
Other:
- board size 326.4 x 201.8 mm -> 92.2 x 65.2 mm

Commit message: Placa de AV 2.0
Connections:
- new net V+: IC1.8
- new net V-: IC1.4
- net +5V: no longer IC1.4
- net GND: no longer IC1.8
Routing:
- net +5V: track 212.4 -> 210.1 mm
Changed lines of the file:
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@@
 <contactref element="C2" pad="1"/>
 <contactref element="X7" pad="3"/>
-<contactref element="IC1" pad="8"/>
 <contactref element="SV8" pad="2"/>
 <contactref element="X1" pad="2"/>
@@
 <via x="130.81635" y="-10.287" extent="1-16" drill="0.8"/>
 <via x="130.81635" y="-14.23035" extent="1-16" drill="0.8"/>
-<wire x1="130.81635" y1="-10.287" x2="130.81635" y2="-14.23035" width="0" layer="19" extent="1-1"/>
+<wire x1="160.344" y1="7.271" x2="181.3941" y2="-6.1722" width="0" layer="19" extent="16-16"/>
+<wire x1="152.724" y1="4.731" x2="160.344" y2="7.271" width="0" layer="19" extent="1-1"/>
+<wire x1="147.415" y1="-3.772" x2="152.724" y2="4.731" width="0" layer="19" extent="1-1"/>
+<wire x1="147.415" y1="-8.744" x2="147.415" y2="-3.772" width="0" layer="19" extent="1-1"/>
+<wire x1="142.3349" y1="2.40015" x2="147.415" y2="-3.772" width="0" layer="19" extent="1-1"/>
+<wire x1="142.5069" y1="12.1728" x2="142.3349" y2="2.40015" width="0" layer="19" extent="1-1"/>
+<wire x1="142.91945" y1="24.003" x2="142.5069" y2="12.1728" width="0" layer="19" extent="1-1"/>
+<wire x1="133.731" y1="24.6888" x2="142.91945" y2="24.003" width="0" layer="19" extent="16-16"/>
+<wire x1="125.4699" y1="24.86035" x2="131.8085" y2="25.33805" width="0" layer="19" extent="16-16"/>
+<wire x1="126.00965" y1="21.2914" x2="125.4699" y2="24.86035" width="0" layer="19" extent="1-1"/>
+<wire x1="119.50725" y1="21.2914" x2="126.00965" y2="21.2914" width="0" layer="19" extent="1-1"/>
+<wire x1="116.04015" y1="25.0319" x2="119.50725" y2="21.2914" width="0" layer="19" extent="1-1"/>
+<wire x1="113.157" y1="20.0274" x2="116.04015" y2="25.0319" width="0" layer="19" extent="1-1"/>
+<wire x1="119.84335" y1="8.78175" x2="119.50725" y2="21.2914" width="0" layer="19" extent="1-1"/>
+<wire x1="112.98535" y1="2.08875" x2="119.84335" y2="8.78175" width="0" layer="19" extent="1-1"/>
+<wire x1="120.01525" y1="-2.3623" x2="112.98535" y2="2.08875" width="0" layer="19" extent="1-1"/>
+<wire x1="113.32825" y1="-9.2263" x2="120.01525" y2="-2.3623" width="0" layer="19" extent="1-1"/>
+<wire x1="130.81635" y1="-10.287" x2="120.01525" y2="-2.3623" width="0" layer="19" extent="1-1"/>
+<wire x1="130.81635" y1="-14.23035" x2="130.81635" y2="-10.287" width="0" layer="19" extent="1-1"/>
+<wire x1="158.4198" y1="-25.1714" x2="147.415" y2="-8.744" width="0" layer="19" extent="1-1"/>
 </signal>
 <signal name="+5V">
@@
 <contactref element="X7" pad="1"/>
 <contactref element="C2" pad="2"/>
-<contactref element="IC1" pad="4"/>
 <contactref element="SV8" pad="1"/>
 <contactref element="X1" pad="1"/>
@@
 <wire x1="181.56555" y1="-13.54455" x2="185.0706" y2="-10.0395" width="0.6096" layer="16"/>
 <wire x1="185.0706" y1="-10.0395" x2="185.0706" y2="-8.57295" width="0.6096" layer="16"/>
-<wire x1="129.921" y1="4.4196" x2="131.50215" y2="6.00075" width="0.6096" layer="16"/>
 <wire x1="131.50215" y1="6.00075" x2="131.50215" y2="7.5438" width="0.6096" layer="16"/>
 <wire x1="131.50215" y1="7.5438" x2="130.81635" y2="8.2296" width="0.6096" layer="16"/>
@@
 </polygon>
 </signal>
+<signal name="V-">
+<contactref element="IC1" pad="4"/>
+</signal>
+<signal name="V+">
+<contactref element="IC1" pad="8"/>
+</signal>
 </signals>
