File: PB01 - Hardware/HW04 - Placa de ECU2 Telemetria/ecu2_telemetria.sch (EAGLE design)
At the start: 26 parts, among them IC1 LM358N, Q2 16MHz, X1 22-23-2021, X5 22-23-2021, X6 22-23-2021, X8 22-23-2031

Commit message: TE#LEMETRIA
Parts:
- removed C1, C4: 100nF, capacitor-wima:C5/2.5
- removed D5: 1N4004, diode:1N4004
- removed D6: 3.3V, diode:ZENER-DIODEDO34-7
- removed OK1: PC817, optocoupler:PC817
- removed R1, R2, R4, R8: 1k, resistor:R-EU_0207/7
- removed R3: 10k, resistor:R-EU_0207/7
- removed R7: 4.7KR, resistor:R-EU_0207/7
- removed SV1: (no value), con-lstb:MA06-1
- removed X6: 22-23-2021, con-molex:22-23-2021
- removed X8: 22-23-2031, con-molex:22-23-2031
- added C7, C8: 100nF, capacitor-wima:C5/2.5
- added D2, D3: 5.0V, diode:ZENER-DIODEDO34-7
- added R10, R12: 1k, resistor:R-EU_0207/7
- added R11, R9: 4.7KR, resistor:R-EU_0207/7
- added X2: COMB 1, con-molex:22-23-2031
- added X3: COMB 2, con-molex:22-23-2031
- added X4: MODULE CAN, con-molex:22-23-2071
- added X7: FORÇA, con-molex:22-23-2031
- C2: device capacitor-wima:C2,5-3 -> capacitor-wima:C5/2.5
- IC1: device linear3:LM358N -> linear:LM358N
- X1: value 22-23-2021 -> DAC; device con-molex:22-23-2021 -> con-molex:22-23-2031
- X5: value 22-23-2021 -> 22-23-2041; device con-molex:22-23-2021 -> con-molex:22-23-2041
- renumbered Q2 to CRISTAL, S1 to BOTÃO
Connections:
- removed net N$1: OK1.A, R1.2, R2.2
- removed net N$2: D5.C, R1.1, R2.1
- removed net N$4: IC1B.-IN, IC1B.OUT, R4.1
- removed net N$7: IC1B.+IN, OK1.EMIT, R3.2
- removed net N$8: D6.C, IC1A.+IN, R7.2
- removed net PA10: IC1A.-IN, IC1A.OUT, R8.1
- removed net RPM_GND: OK1.C, X1-2.S
- removed net RPM_IN: D5.A, X1-1.S
- removed net RPM_OUT: C1.2, R4.2, ZIC1.(INT0)PD2
- removed net VEL_IN: R7.1, X8-2.S
- removed net VEL_OUT: C4.2, R8.2, ZIC1.(INT1)PD3
- new net N$12: IC1A.-IN, IC1A.OUT, R10.1
- new net N$13: D3.C, IC1B.+IN, R11.2
- new net N$14: IC1B.-IN, IC1B.OUT, R12.1
- new net N$3: X1-3.S, ZIC1.(AIN0)PD6
- new net N$5: D2.C, IC1A.+IN, R9.2
- new net SCL: X5-3.S, ZIC1.(ADC5)PC5
- new net SDA: X5-4.S, ZIC1.(ADC4)PC4
- new net VEL1_IN: R9.1, X3-2.S
- new net VEL1_OUT: C7.2, R10.2, ZIC1.(INT1)PD3
- new net VEL2_IN: R11.1, X2-2.S
- new net VEL2_OUT: C8.2, R12.2, ZIC1.(INT0)PD2
- net +12V: now also X2-1.S, X3-1.S, X7-2.S; no longer X6-1.S, X8-1.S
- net +5V: now also IC1P.V-, X1-1.S, X4-7.S, X7-1.S; no longer IC1P.V+, OK1.COL, SV1.5
- net GND: now also C7.1, C8.1, D2.A, D3.A, IC1P.V+, X1-2.S, X2-3.S, X3-3.S, X4-6.S, X7-3.S; no longer C1.1, C4.1, D6.A, IC1P.V-, R3.1, SV1.6, X6-2.S, X8-3.S
- net MISO: now also X4-4.S; no longer SV1.4
- net MOSI: now also X4-3.S; no longer SV1.3
- net SCK: now also X4-2.S; no longer SV1.2
- net SS: now also X4-5.S; no longer SV1.1
Other:
- moved on the sheet: C2, IC1A, IC1B, SV8, X1-1, X1-2, X5-1, X5-2

Commit message: Placa de AV 2.0
Connections:
- net +5V: no longer IC1P.V-
- net GND: no longer IC1P.V+
Changed lines of the file:
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@@
 <grid distance="0.05" unitdist="inch" unit="inch" style="lines" multiple="1" display="no" altdistance="0.01" altunitdist="inch" altunit="inch"/>
 <layers>
-<layer number="1" name="Top" color="4" fill="1" visible="yes" active="no"/>
-<layer number="2" name="Route2" color="1" fill="3" visible="yes" active="no"/>
-<layer number="3" name="Route3" color="4" fill="3" visible="yes" active="no"/>
-<layer number="4" name="Route4" color="1" fill="4" visible="yes" active="no"/>
-<layer number="5" name="Route5" color="4" fill="4" visible="yes" active="no"/>
-<layer number="6" name="Route6" color="1" fill="8" visible="yes" active="no"/>
-<layer number="7" name="Route7" color="4" fill="8" visible="yes" active="no"/>
-<layer number="8" name="Route8" color="1" fill="2" visible="yes" active="no"/>
-<layer number="9" name="Route9" color="4" fill="2" visible="yes" active="no"/>
-<layer number="10" name="Route10" color="1" fill="7" visible="yes" active="no"/>
-<layer number="11" name="Route11" color="4" fill="7" visible="yes" active="no"/>
-<layer number="12" name="Route12" color="1" fill="5" visible="yes" active="no"/>
-<layer number="13" name="Route13" color="4" fill="5" visible="yes" active="no"/>
-<layer number="14" name="Route14" color="1" fill="6" visible="yes" active="no"/>
-<layer number="15" name="Route15" color="4" fill="6" visible="yes" active="no"/>
-<layer number="16" name="Bottom" color="1" fill="1" visible="yes" active="no"/>
-<layer number="17" name="Pads" color="2" fill="1" visible="yes" active="no"/>
-<layer number="18" name="Vias" color="2" fill="1" visible="yes" active="no"/>
-<layer number="19" name="Unrouted" color="6" fill="1" visible="yes" active="no"/>
-<layer number="20" name="Dimension" color="24" fill="1" visible="yes" active="no"/>
-<layer number="21" name="tPlace" color="7" fill="1" visible="yes" active="no"/>
-<layer number="22" name="bPlace" color="7" fill="1" visible="yes" active="no"/>
-<layer number="23" name="tOrigins" color="15" fill="1" visible="yes" active="no"/>
-<layer number="24" name="bOrigins" color="15" fill="1" visible="yes" active="no"/>
-<layer number="25" name="tNames" color="7" fill="1" visible="yes" active="no"/>
-<layer number="26" name="bNames" color="7" fill="1" visible="yes" active="no"/>
-<layer number="27" name="tValues" color="7" fill="1" visible="yes" active="no"/>
-<layer number="28" name="bValues" color="7" fill="1" visible="yes" active="no"/>
+<layer number="1" name="Top" color="4" fill="1" visible="no" active="no"/>
+<layer number="2" name="Route2" color="1" fill="3" visible="no" active="no"/>
+<layer number="3" name="Route3" color="4" fill="3" visible="no" active="no"/>
+<layer number="4" name="Route4" color="1" fill="4" visible="no" active="no"/>
+<layer number="5" name="Route5" color="4" fill="4" visible="no" active="no"/>
+<layer number="6" name="Route6" color="1" fill="8" visible="no" active="no"/>
+<layer number="7" name="Route7" color="4" fill="8" visible="no" active="no"/>
+<layer number="8" name="Route8" color="1" fill="2" visible="no" active="no"/>
+<layer number="9" name="Route9" color="4" fill="2" visible="no" active="no"/>
+<layer number="10" name="Route10" color="1" fill="7" visible="no" active="no"/>
+<layer number="11" name="Route11" color="4" fill="7" visible="no" active="no"/>
+<layer number="12" name="Route12" color="1" fill="5" visible="no" active="no"/>
+<layer number="13" name="Route13" color="4" fill="5" visible="no" active="no"/>
+<layer number="14" name="Route14" color="1" fill="6" visible="no" active="no"/>
+<layer number="15" name="Route15" color="4" fill="6" visible="no" active="no"/>
+<layer number="16" name="Bottom" color="1" fill="1" visible="no" active="no"/>
+<layer number="17" name="Pads" color="2" fill="1" visible="no" active="no"/>
+<layer number="18" name="Vias" color="2" fill="1" visible="no" active="no"/>
+<layer number="19" name="Unrouted" color="6" fill="1" visible="no" active="no"/>
+<layer number="20" name="Dimension" color="24" fill="1" visible="no" active="no"/>
+<layer number="21" name="tPlace" color="7" fill="1" visible="no" active="no"/>
+<layer number="22" name="bPlace" color="7" fill="1" visible="no" active="no"/>
+<layer number="23" name="tOrigins" color="15" fill="1" visible="no" active="no"/>
+<layer number="24" name="bOrigins" color="15" fill="1" visible="no" active="no"/>
+<layer number="25" name="tNames" color="7" fill="1" visible="no" active="no"/>
+<layer number="26" name="bNames" color="7" fill="1" visible="no" active="no"/>
+<layer number="27" name="tValues" color="7" fill="1" visible="no" active="no"/>
+<layer number="28" name="bValues" color="7" fill="1" visible="no" active="no"/>
 <layer number="29" name="tStop" color="7" fill="3" visible="no" active="no"/>
 <layer number="30" name="bStop" color="7" fill="6" visible="no" active="no"/>
@@
 <layer number="35" name="tGlue" color="7" fill="4" visible="no" active="no"/>
 <layer number="36" name="bGlue" color="7" fill="5" visible="no" active="no"/>
-<layer number="37" name="tTest" color="7" fill="1" visible="yes" active="no"/>
-<layer number="38" name="bTest" color="7" fill="1" visible="yes" active="no"/>
+<layer number="37" name="tTest" color="7" fill="1" visible="no" active="no"/>
+<layer number="38" name="bTest" color="7" fill="1" visible="no" active="no"/>
 <layer number="39" name="tKeepout" color="4" fill="11" visible="no" active="no"/>
 <layer number="40" name="bKeepout" color="1" fill="11" visible="no" active="no"/>
@@
 <layer number="44" name="Drills" color="7" fill="1" visible="no" active="no"/>
 <layer number="45" name="Holes" color="7" fill="1" visible="no" active="no"/>
-<layer number="46" name="Milling" color="3" fill="1" visible="yes" active="no"/>
-<layer number="47" name="Measures" color="7" fill="1" visible="yes" active="no"/>
-<layer number="48" name="Document" color="7" fill="1" visible="yes" active="no"/>
-<layer number="49" name="Reference" color="7" fill="1" visible="yes" active="no"/>
-<layer number="50" name="dxf" color="7" fill="1" visible="yes" active="no"/>
-<layer number="51" name="tDocu" color="7" fill="1" visible="yes" active="no"/>
-<layer number="52" name="bDocu" color="7" fill="1" visible="yes" active="no"/>
-<layer number="53" name="tGND_GNDA" color="7" fill="9" visible="yes" active="no"/>
-<layer number="54" name="bGND_GNDA" color="1" fill="9" visible="yes" active="no"/>
-<layer number="56" name="wert" color="3" fill="1" visible="yes" active="no"/>
-<layer number="57" name="tCAD" color="7" fill="1" visible="yes" active="no"/>
-<layer number="59" name="tCarbon" color="7" fill="1" visible="yes" active="no"/>
-<layer number="60" name="bCarbon" color="7" fill="1" visible="yes" active="no"/>
+<layer number="46" name="Milling" color="3" fill="1" visible="no" active="no"/>
+<layer number="47" name="Measures" color="7" fill="1" visible="no" active="no"/>
+<layer number="48" name="Document" color="7" fill="1" visible="no" active="no"/>
+<layer number="49" name="Reference" color="7" fill="1" visible="no" active="no"/>
+<layer number="50" name="dxf" color="7" fill="1" visible="no" active="no"/>
+<layer number="51" name="tDocu" color="7" fill="1" visible="no" active="no"/>
+<layer number="52" name="bDocu" color="7" fill="1" visible="no" active="no"/>
+<layer number="53" name="tGND_GNDA" color="7" fill="9" visible="no" active="no"/>
+<layer number="54" name="bGND_GNDA" color="1" fill="9" visible="no" active="no"/>
+<layer number="56" name="wert" color="3" fill="1" visible="no" active="no"/>
+<layer number="57" name="tCAD" color="7" fill="1" visible="no" active="no"/>
+<layer number="59" name="tCarbon" color="7" fill="1" visible="no" active="no"/>
+<layer number="60" name="bCarbon" color="7" fill="1" visible="no" active="no"/>
 <layer number="88" name="SimResults" color="9" fill="1" visible="yes" active="yes"/>
 <layer number="89" name="SimProbes" color="9" fill="1" visible="yes" active="yes"/>
@@
 <instance part="IC1" gate="A" x="-95.25" y="83.82"/>
 <instance part="IC1" gate="B" x="-99.06" y="38.1"/>
-<instance part="IC1" gate="P" x="-173.99" y="69.85" rot="R270"/>
+<instance part="IC1" gate="P" x="-173.99" y="72.39" rot="R90"/>
 <instance part="SV8" gate="G$1" x="123.19" y="130.81" rot="R180"/>
 <instance part="P+8" gate="1" x="113.03" y="142.24" smashed="yes">
@@
 <wire x1="-166.37" y1="68.58" x2="-160.02" y2="68.58" width="0.1524" layer="91"/>
 <pinref part="C2" gate="G$1" pin="1"/>
-<pinref part="IC1" gate="P" pin="V+"/>
-<wire x1="-166.37" y1="69.85" x2="-166.37" y2="68.58" width="0.1524" layer="91"/>
-<junction x="-166.37" y="68.58"/>
 </segment>
 <segment>
@@
 <wire x1="-185.42" y1="68.58" x2="-185.42" y2="71.12" width="0.1524" layer="91"/>
 <pinref part="C2" gate="G$1" pin="2"/>
-<pinref part="IC1" gate="P" pin="V-"/>
-<wire x1="-181.61" y1="69.85" x2="-181.61" y2="68.58" width="0.1524" layer="91"/>
-<junction x="-181.61" y="68.58"/>
-</segment>
-<segment>
+</segment>
+<segment>
