File: PB01 - Hardware/HW06 - Placa de teste AV 2.0/Schematic/placa_teste_av.brd (EAGLE design)
At the start: 326.4 x 201.8 mm, 24 parts, among them IC1 LM358N, X1 DAC, X2 COMB 1, X3 COMB 2, X4 MODULE CAN, X5 22-23-2041, X7 FORÇA

Commit message: Placa de AV 2.0
Parts:
- removed BOTÃO: (no value), switch-omron:B3F-10XX
- removed C2, C8: 100nF, capacitor-wima:C5B2.5
- removed CRISTAL: 16MHz, special:QS
- removed D3: 5.0V, diode:DO34Z7
- removed IC1: LM358N, linear:DIL08
- removed R11: 4.7KR, resistor:0207/7
- removed R12: 1k, resistor:0207/7
- removed SV8: (no value), con-lstb:MA05-1
- removed X5: 22-23-2041, con-molex:22-23-2041
- added C1, C11: (no value), capacitor-wima:C5B2.5
- added C4: (no value), resistor:C025-024X044
- added D5: 1N4004, diode:DO41-10
- added D6: 3.3V, diode:DO34Z7
- added IC2: LM324N, linear:DIL14
- added JP1, JP2, JP3: (no value), pinhead:1X01
- added OK1: PC817, optocoupler:DIL04
- added Q2: 16MHz, special:QS
- added R1, R2, R4, R8: 1k, resistor:0207/7
- added R3: 10k, resistor:0207/7
- added R7: 4.7KR, resistor:0207/7
- added S1: (no value), switch-omron:B3F-10XX
- added SV2: (no value), con-lstb:MA05-1
- added X10, X11: 22-23-2021, con-molex:22-23-2021
- added X8: 22-23-2031, con-molex:22-23-2031
- C3: value 100nF -> (none); device capacitor-wima:C5B2.5 -> resistor:C025-024X044
- C5, C6: value 22pF -> (none)
- C7: value 100nF -> (none)
- X1: value DAC -> 22-23-2021; device con-molex:22-23-2031 -> con-molex:22-23-2021
- X2: value COMB 1 -> 22-23-2041; device con-molex:22-23-2031 -> con-molex:22-23-2041
- X4: value MODULE CAN -> DAC; device con-molex:22-23-2071 -> con-molex:22-23-2031
- X7: value FORÇA -> 22-23-2031
- moved X4 95.1 mm to (84.0, -26.1)
- moved X1 91.9 mm to (41.8, 14.7), turned to 180 degrees
- moved R10 82.3 mm to (69.4, -17.7)
- moved C7 82.2 mm to (69.4, -20.7), turned to 180 degrees
- moved C5 76.0 mm to (69.3, -11.1), turned to 180 degrees
- moved C6 75.9 mm to (69.3, -1.89), turned to 180 degrees
- moved ZIC1 63.5 mm to (95.0, -9.77)
- moved R9 62.0 mm to (63.1, 5.49), turned to 180 degrees
- moved D2 58.9 mm to (63.1, 9.09), turned to 0 degrees
- moved C3 57.3 mm to (79.2, -12.2), turned to 0 degrees
- moved X3 54.1 mm to (63.4, 14.9), turned to 180 degrees
- moved R5 31.9 mm to (91.2, 10.5), turned to 0 degrees
- moved X2 12.5 mm to (116.8, 16.3), turned to 0 degrees
- moved X7 11.3 mm to (102.2, 14.9), turned to 0 degrees
Connections:
- net VEL1_IN renamed COMB1_IN
- removed net IO8: SV8.3, ZIC1.14
- removed net IO9: SV8.4, ZIC1.15
- removed net MISO: X4.4, ZIC1.18
- removed net MOSI: X4.3, ZIC1.17
- removed net N$13: D3.C, IC1.5, R11.2
- removed net N$14: IC1.6, IC1.7, R12.1
- removed net N$6: SV8.5
- removed net SCK: X4.2, ZIC1.19
- removed net SS: X4.5, ZIC1.16
- removed net VEL1_OUT: C7.2, R10.2, ZIC1.5
- removed net VEL2_IN: R11.1, X2.2
- removed net VEL2_OUT: C8.2, R12.2, ZIC1.4
- new net COMB1_OUT: C7.1, JP3.1, R10.2, ZIC1.6
- new net IO1: SV2.3, X11.2, ZIC1.14
- new net IO2: SV2.4, X11.1, ZIC1.15
- new net N$1: OK1.1, R1.2, R2.2
- new net N$10: X4.3, ZIC1.12
- new net N$2: D5.C, R1.1, R2.1
- new net N$4: IC2.1, IC2.2, R4.1
- new net N$7: IC2.3, OK1.3, R3.2
- new net N$8: D6.C, IC2.12, R7.2
- new net PA10: IC2.13, IC2.14, R8.1
- new net RPM_GND: OK1.2, X1.2
- new net RPM_IN: D5.A, X1.1
- new net RPM_OUT: C5.1, JP1.1, R4.2, ZIC1.5
- new net VEL_IN: R7.1, X8.2
- new net VEL_OUT: C6.1, JP2.1, R8.2, ZIC1.4
- net +12V: now also X3.3, X8.1; no longer X2.1, X3.1
- net +5V: now also C1.1, C11.1, IC2.4, OK1.4, SV2.1, X2.1, X4.1; no longer C2.2, C3.2, IC1.4, SV8.1, X1.1, X4.7, X5.1
- net GND: now also C1.2, C11.2, C4.1, C7.2, D6.A, IC2.11, R3.1, S1.1, S1.2, SV2.2, X2.2, X3.1, X4.2, X8.3; no longer BOTÃO.1, BOTÃO.2, C2.1, C7.1, C8.1, D3.A, IC1.8, SV8.2, X1.2, X2.3, X3.3, X4.6, X5.2
- net N$12: now also IC2.8, IC2.9; no longer IC1.1, IC1.2
- net N$3: now also SV2.5; no longer X1.3, ZIC1.12
- net N$5: now also IC2.10; no longer IC1.3
- net N$9: now also S1.3, S1.4; no longer BOTÃO.3, BOTÃO.4
- net SCL: now also X10.1, X2.3; no longer X5.3
- net SDA: now also X10.2, X2.4; no longer X5.4
- net XTAL1: now also C3.2, Q2.2; no longer C6.1, CRISTAL.2
- net XTAL2: now also C4.2, Q2.1; no longer C5.1, CRISTAL.1
Routing:
- net +5V: track 28.6 -> 218.9 mm
- net +12V: track 0.00 -> 53.4 mm
- net IO1: track 0.00 -> 45.7 mm
- net N$5: track 0.00 -> 34.6 mm
- net SDA: track 0.00 -> 32.1 mm
- net IO2: track 0.00 -> 31.2 mm
- net COMB1_OUT: track 0.00 -> 29.0 mm
- net SCL: track 0.00 -> 27.2 mm
- net N$8: track 0.00 -> 24.7 mm
- net RPM_OUT: track 0.00 -> 24.7 mm
- net VEL_OUT: track 0.00 -> 23.3 mm
- net N$7: track 0.00 -> 21.7 mm
- net N$4: track 0.00 -> 20.3 mm
- net XTAL1: track 29.2 -> 11.3 mm
- net N$1: track 0.00 -> 15.2 mm
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- added copper zone on layer 16, net GND
- removed copper zone on layer 16, net MODULE_CAN
- removed copper zone on layer 16, net N$1
Other:
- board size 326.4 x 201.8 mm -> 96 x 50.1 mm
- board text removed: "Design by: Matheus Torres Rocha"
- board text removed: "Equipe ParahyBaja ECU1"

Commit message: teste de av 2.0
Parts:
- moved X10 5.55 mm to (124.9, 9.18)
- moved SV2 1.28 mm to (112.0, -24.1)
Routing:
- net +5V: track 218.9 -> 246.9 mm
- net SDA: track 32.1 -> 41.3 mm
- net N$1: track 15.2 -> 24.3 mm
- net XTAL2: track 11.2 -> 18.4 mm
- net SCL: track 27.2 -> 34.0 mm
- net N$2: track 7.20 -> 12.3 mm
- net VEL_OUT: track 23.3 -> 26.4 mm
- net +12V: track 53.4 -> 51.1 mm
- net IO1: track 45.7 -> 44.2 mm
- net IO2: track 31.2 -> 30.2 mm
