File: PB01 - Hardware/HW08 - Placa ECU2 NAC20/ecu2.brd (EAGLE design)
At the start: 92.9 x 54.9 mm, 18 parts, among them IC1 LM358N, X4 MODULE CAN

Commit message: ECU2_2020
Parts:
- added LEDS: FORÇA, con-molex:22-23-2031
Connections:
- new net LEDS: LEDS.2, U$1.D6
- net +5V: now also LEDS.1
- net GND: now also LEDS.3
Routing:
- net LEDS: track 0.00 -> 25.0 mm
- net RST: track 58.5 -> 57.6 mm
- net +5V: track 149.9 -> 149.2 mm
